Commit message: Hook on the uuv

File: uuv/uuv.urdf (robot description, URDF)
Before this commit: robot UUV, 1 links, 0 joints
Links:
- added link origin_black; visual mesh filename=hook_black.stl
- added link origin_steel; visual mesh filename=hook_steel.stl
- added link origin_white; visual mesh filename=hook_white.stl
- link origin: geometry visual mesh filename=package://uuv/UUV v1.stl
Joints:
- added joint hook_joint: type fixed, parent origin, child origin_white
- added joint origin_1: type fixed, parent origin_white, child origin_black
- added joint origin_2: type fixed, parent origin_black, child origin_steel
