Commit message: Added triad example

File: bpl_bravo_description/urdf/bravo_7_example_with_camera.urdf (robot description, URDF)
Before this commit: robot bravo_7_example, 28 links, 27 joints
Links:
- link camera_end_link: geometry collision cylinder length=0.01 radius=0.001; visual cylinder length=0.01 radius=0.001
Joints:
- joint camera_end_joint: origin xyz=0 0 0 rpy=0 0 0 -> xyz=0.01326 0.05195 +0.02 rpy=0 0 0

Commit message: End effector visualisation and end effector link

File: bpl_bravo_description/urdf/bravo_7_example_with_camera.urdf (robot description, URDF)
Before this commit: robot bravo_7_example, 28 links, 27 joints
Links:
- added link end_effector_link; visual cylinder length=0.01 radius=0.001
Joints:
- added joint end_effector_joint: type fixed, parent bravo_1028_end_link, child end_effector_link, origin xyz=0.10 0.00 0.00 rpy=0 0 0

Commit message: Hack together wrist camera view.

File: bpl_bravo_description/urdf/bravo_7_example_with_camera.urdf (robot description, URDF)
Before this commit: robot bravo_7_example, 29 links, 28 joints
Joints:
- joint camera_end_joint: origin xyz=0.01326 0.05195 +0.02 rpy=0 0 0 -> xyz=0.01326 0.05195 +0.02 rpy=3.14 0 0

Commit message: makde bravo axis d continious. Setup initial position

File: bpl_bravo_description/urdf/bravo_7_example_with_camera.urdf (robot description, URDF)
Before this commit: robot bravo_7_example, 29 links, 28 joints
Joints:
- joint bravo_axis_d: limit lower=0 upper=6.2 effort=0 velocity=0 -> (none); type revolute -> continuous

Commit message: Jaws working

File: bpl_bravo_description/urdf/bravo_7_example_with_camera.urdf (robot description, URDF)
Before this commit: robot bravo_7_example, 29 links, 28 joints
Links:
- link end_effector_link: geometry visual cylinder length=0.01 radius=0.00001
