Commit message: rectangle

File: sphereG.urdf (robot description, URDF)
Before this commit: robot myfirst, 1 links, 0 joints
Links:
- link base_link: geometry visual sphere radius=0.002

File: sphereR.urdf (robot description, URDF)
Before this commit: robot myfirst, 1 links, 0 joints
Links:
- link base_link: geometry visual sphere radius=0.002

Commit message: state fix

File: sphereG.urdf (robot description, URDF)
Before this commit: robot myfirst, 1 links, 0 joints
Links:
- link base_link: geometry visual sphere radius=0.02

File: sphereR.urdf (robot description, URDF)
Before this commit: robot myfirst, 1 links, 0 joints
Links:
- link base_link: geometry visual sphere radius=0.02
